Commit message: Fix urdf mesh file paths

File: dm_arm_description/urdf/dm_arm.urdf (robot description, URDF)
Before this commit: robot dm_arm, 11 links, 10 joints
Links:
- link base_link: geometry collision mesh filename=package://dm_arm_description/meshes/base_link.STL; visual mesh filename=package://dm_arm_description/meshes/base_link.STL
- link link1: geometry collision mesh filename=package://dm_arm_description/meshes/link1.STL; visual mesh filename=package://dm_arm_description/meshes/link1.STL
- link link2: geometry collision mesh filename=package://dm_arm_description/meshes/link2.STL; visual mesh filename=package://dm_arm_description/meshes/link2.STL
- link link3: geometry collision mesh filename=package://dm_arm_description/meshes/link3.STL; visual mesh filename=package://dm_arm_description/meshes/link3.STL
- link link4: geometry collision mesh filename=package://dm_arm_description/meshes/link4.STL; visual mesh filename=package://dm_arm_description/meshes/link4.STL
- link link5: geometry collision mesh filename=package://dm_arm_description/meshes/link5.STL; visual mesh filename=package://dm_arm_description/meshes/link5.STL
- link link6: geometry collision mesh filename=package://dm_arm_description/meshes/link6.STL; visual mesh filename=package://dm_arm_description/meshes/link6.STL
- link link7_1: geometry collision mesh filename=package://dm_arm_description/meshes/link7_1.STL; visual mesh filename=package://dm_arm_description/meshes/link7_1.STL
- link link7_2: geometry collision mesh filename=package://dm_arm_description/meshes/link7_2.STL; visual mesh filename=package://dm_arm_description/meshes/link7_2.STL
